Commit message: fix urdf scale

File: ycb_assets/002_master_chef_can.urdf (robot description, URDF)
Before this commit: robot 002_master_chef_can, 1 links, 0 joints
Links:
- link _name: geometry collision mesh filename=002_master_chef_can/google_16k/textured_vhacd.obj scale=1 1 1; visual mesh filename=002_master_chef_can/google_16k/textured.obj scale=1 1 1

File: ycb_assets/003_cracker_box.urdf (robot description, URDF)
Before this commit: robot 003_cracker_box, 1 links, 0 joints
Links:
- link _name: geometry collision mesh filename=003_cracker_box/google_16k/textured_vhacd.obj scale=1 1 1; visual mesh filename=003_cracker_box/google_16k/textured.obj scale=1 1 1

File: ycb_assets/004_sugar_box.urdf (robot description, URDF)
Before this commit: robot 004_sugar_box, 1 links, 0 joints
Links:
- link _name: geometry collision mesh filename=004_sugar_box/google_16k/textured_vhacd.obj scale=1 1 1; visual mesh filename=004_sugar_box/google_16k/textured.obj scale=1 1 1

File: ycb_assets/005_tomato_soup_can.urdf (robot description, URDF)
Before this commit: robot 005_tomato_soup_can, 1 links, 0 joints
Links:
- link _name: geometry collision mesh filename=005_tomato_soup_can/google_16k/textured_vhacd.obj scale=1 1 1; visual mesh filename=005_tomato_soup_can/google_16k/textured.obj scale=1 1 1

File: ycb_assets/006_mustard_bottle.urdf (robot description, URDF)
Before this commit: robot 006_mustard_bottle, 1 links, 0 joints
Links:
- link _name: geometry collision mesh filename=006_mustard_bottle/google_16k/textured_vhacd.obj scale=1 1 1; visual mesh filename=006_mustard_bottle/google_16k/textured.obj scale=1 1 1

File: ycb_assets/007_tuna_fish_can.urdf (robot description, URDF)
Before this commit: robot 007_tuna_fish_can, 1 links, 0 joints
Links:
- link _name: geometry collision mesh filename=007_tuna_fish_can/google_16k/textured_vhacd.obj scale=1 1 1; visual mesh filename=007_tuna_fish_can/google_16k/textured.obj scale=1 1 1

File: ycb_assets/008_pudding_box.urdf (robot description, URDF)
Before this commit: robot 008_pudding_box, 1 links, 0 joints
Links:
- link _name: geometry collision mesh filename=008_pudding_box/google_16k/textured_vhacd.obj scale=1 1 1; visual mesh filename=008_pudding_box/google_16k/textured.obj scale=1 1 1

File: ycb_assets/009_gelatin_box.urdf (robot description, URDF)
Before this commit: robot 009_gelatin_box, 1 links, 0 joints
Links:
- link _name: geometry collision mesh filename=009_gelatin_box/google_16k/textured_vhacd.obj scale=1 1 1; visual mesh filename=009_gelatin_box/google_16k/textured.obj scale=1 1 1

File: ycb_assets/010_potted_meat_can.urdf (robot description, URDF)
Before this commit: robot 010_potted_meat_can, 1 links, 0 joints
Links:
- link _name: geometry collision mesh filename=010_potted_meat_can/google_16k/textured_vhacd.obj scale=1 1 1; visual mesh filename=010_potted_meat_can/google_16k/textured.obj scale=1 1 1

File: ycb_assets/011_banana.urdf (robot description, URDF)
Before this commit: robot 011_banana, 1 links, 0 joints
Links:
- link _name: geometry collision mesh filename=011_banana/google_16k/textured_vhacd.obj scale=1 1 1; visual mesh filename=011_banana/google_16k/textured.obj scale=1 1 1

File: ycb_assets/012_strawberry.urdf (robot description, URDF)
Before this commit: robot 012_strawberry, 1 links, 0 joints
Links:
- link _name: geometry collision mesh filename=012_strawberry/google_16k/textured_vhacd.obj scale=1 1 1; visual mesh filename=012_strawberry/google_16k/textured.obj scale=1 1 1

File: ycb_assets/013_apple.urdf (robot description, URDF)
Before this commit: robot 013_apple, 1 links, 0 joints
Links:
- link _name: geometry collision mesh filename=013_apple/google_16k/textured_vhacd.obj scale=1 1 1; visual mesh filename=013_apple/google_16k/textured.obj scale=1 1 1

File: ycb_assets/014_lemon.urdf (robot description, URDF)
Before this commit: robot 014_lemon, 1 links, 0 joints
Links:
- link _name: geometry collision mesh filename=014_lemon/google_16k/textured_vhacd.obj scale=1 1 1; visual mesh filename=014_lemon/google_16k/textured.obj scale=1 1 1

File: ycb_assets/015_peach.urdf (robot description, URDF)
Before this commit: robot 015_peach, 1 links, 0 joints
Links:
- link _name: geometry collision mesh filename=015_peach/google_16k/textured_vhacd.obj scale=1 1 1; visual mesh filename=015_peach/google_16k/textured.obj scale=1 1 1

File: ycb_assets/016_pear.urdf (robot description, URDF)
Before this commit: robot 016_pear, 1 links, 0 joints
Links:
- link _name: geometry collision mesh filename=016_pear/google_16k/textured_vhacd.obj scale=1 1 1; visual mesh filename=016_pear/google_16k/textured.obj scale=1 1 1

File: ycb_assets/017_orange.urdf (robot description, URDF)
Before this commit: robot 017_orange, 1 links, 0 joints
Links:
- link _name: geometry collision mesh filename=017_orange/google_16k/textured_vhacd.obj scale=1 1 1; visual mesh filename=017_orange/google_16k/textured.obj scale=1 1 1

File: ycb_assets/018_plum.urdf (robot description, URDF)
Before this commit: robot 018_plum, 1 links, 0 joints
Links:
- link _name: geometry collision mesh filename=018_plum/google_16k/textured_vhacd.obj scale=1 1 1; visual mesh filename=018_plum/google_16k/textured.obj scale=1 1 1

File: ycb_assets/019_pitcher_base.urdf (robot description, URDF)
Before this commit: robot 019_pitcher_base, 1 links, 0 joints
Links:
- link _name: geometry collision mesh filename=019_pitcher_base/google_16k/textured_vhacd.obj scale=1 1 1; visual mesh filename=019_pitcher_base/google_16k/textured.obj scale=1 1 1

File: ycb_assets/021_bleach_cleanser.urdf (robot description, URDF)
Before this commit: robot 021_bleach_cleanser, 1 links, 0 joints
Links:
- link _name: geometry collision mesh filename=021_bleach_cleanser/google_16k/textured_vhacd.obj scale=1 1 1; visual mesh filename=021_bleach_cleanser/google_16k/textured.obj scale=1 1 1

File: ycb_assets/022_windex_bottle.urdf (robot description, URDF)
Before this commit: robot 022_windex_bottle, 1 links, 0 joints
Links:
- link _name: geometry collision mesh filename=022_windex_bottle/google_16k/textured_vhacd.obj scale=1 1 1; visual mesh filename=022_windex_bottle/google_16k/textured.obj scale=1 1 1
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